File: 555timersolarcar.kicad_sch (KiCad schematic)
At the start: 11 parts, among them J1 Conn_01x03_Female, J2 Conn_01x02_Female, Q1 Q_NMOS_DGS, U1 NE555D

Commit message: Add files via upload
Parts:
- removed C1: 10uF, Capacitor_SMD:C_0805_2012Metric_Pad1.18x1.45mm_HandSolder, symbol Device:C
- added C1: 100uF, Capacitor_Tantalum_SMD:CP_EIA-7360-38_Kemet-E_Pad2.25x4.25mm_HandSolder, symbol Device:C_Polarized_Small_US
- R3: value 0 -> 10k
- R4: value 5k -> 20k
Connections:
- net GND: now also C1.2
- net at R4.2, U1.2 (TR), U1.6 (THR): now also C1.1
Changed lines of the file:
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@@
+    (stroke (width 0) (type default) (color 0 0 0 0))
+  )
+  (wire (pts (xy 158.75 125.73) (xy 158.75 128.27))
     (stroke (width 0) (type default) (color 0 0 0 0))
   )
@@
     (pin "1")
   )
-  (symbol (lib_id "Device:C") (at 158.75 124.46 0) (unit 1)
-    (in_bom yes) (on_board yes) (fields_autoplaced)
-    (property "Reference" "C1" (id 0) (at 162.56 123.1899 0)
-      (effects (font (size 1.27 1.27)) (justify left))
-    )
-    (property "Value" "10uF" (id 1) (at 162.56 125.7299 0)
-      (effects (font (size 1.27 1.27)) (justify left))
-    )
-    (property "Footprint" "Capacitor_SMD:C_0805_2012Metric_Pad1.18x1.45mm_HandSolder" (id 2) (at 159.7152 128.27 0)
-      (effects (font (size 1.27 1.27)) hide)
-    )
-    (property "Datasheet" "~" (id 3) (at 158.75 124.46 0)
-      (effects (font (size 1.27 1.27)) hide)
-    )
-    (pin "1")
-    (pin "2")
-  )
   (symbol (lib_id "Device:R_Small_US") (at 158.75 110.49 0) (unit 1)
     (in_bom yes) (on_board yes) (fields_autoplaced)
@@
       (effects (font (size 1.27 1.27)) (justify left))
     )
-    (property "Value" "5k" (id 1) (at 161.29 111.7599 0)
+    (property "Value" "20k" (id 1) (at 161.29 111.7599 0)
       (effects (font (size 1.27 1.27)) (justify left))
     )
@@
       (effects (font (size 1.27 1.27)) (justify left))
     )
-    (property "Value" "0" (id 1) (at 161.29 101.5999 0)
+    (property "Value" "10k" (id 1) (at 161.29 101.5999 0)
       (effects (font (size 1.27 1.27)) (justify left))
     )
@@
     )
     (property "Datasheet" "~" (id 3) (at 96.52 97.79 0)
+      (effects (font (size 1.27 1.27)) hide)
+    )
+    (pin "1")
+    (pin "2")
+  )
+  (symbol (lib_id "Device:C_Polarized_Small_US") (at 158.75 123.19 0) (unit 1)
+    (in_bom yes) (on_board yes) (fields_autoplaced)
+    (property "Reference" "C1" (id 0) (at 161.29 121.4881 0)
+      (effects (font (size 1.27 1.27)) (justify left))
+    )
+    (property "Value" "100uF" (id 1) (at 161.29 124.0281 0)
+      (effects (font (size 1.27 1.27)) (justify left))
+    )
+    (property "Footprint" "Capacitor_Tantalum_SMD:CP_EIA-7360-38_Kemet-E_Pad2.25x4.25mm_HandSolder" (id 2) (at 158.75 123.19 0)
+      (effects (font (size 1.27 1.27)) hide)
+    )
+    (property "Datasheet" "~" (id 3) (at 158.75 123.19 0)
       (effects (font (size 1.27 1.27)) hide)
     )
@@
       (reference "#PWR09") (unit 1) (value "+12V") (footprint "")
     )
-    (path "/1751034d-5b7a-457d-b8d0-b5231faa1305"
-      (reference "C1") (unit 1) (value "10uF") (footprint "Capacitor_SMD:C_0805_2012Metric_Pad1.18x1.45mm_HandSolder")
+    (path "/a854696b-b814-4e59-916e-67b8991af0fb"
+      (reference "C1") (unit 1) (value "100uF") (footprint "Capacitor_Tantalum_SMD:CP_EIA-7360-38_Kemet-E_Pad2.25x4.25mm_HandSolder")
     )
     (path "/da0f875d-87f1-4971-a25e-e3eeda8d4d52"
@@
     )
     (path "/48511ee3-0e04-49a5-b2cc-804319b45a20"
-      (reference "R3") (unit 1) (value "0") (footprint "Resistor_SMD:R_0805_2012Metric_Pad1.20x1.40mm_HandSolder")
+      (reference "R3") (unit 1) (value "10k") (footprint "Resistor_SMD:R_0805_2012Metric_Pad1.20x1.40mm_HandSolder")
     )
     (path "/2bdba834-0ed8-4699-8238-8222e5e8b940"
-      (reference "R4") (unit 1) (value "5k") (footprint "Resistor_SMD:R_0805_2012Metric_Pad1.20x1.40mm_HandSolder")
+      (reference "R4") (unit 1) (value "20k") (footprint "Resistor_SMD:R_0805_2012Metric_Pad1.20x1.40mm_HandSolder")
     )
     (path "/80d4696e-d7fa-4fd4-bde5-bd5cf2a96ac7"
