File: 555timersolarcarturnsig.kicad_pcb (KiCad board)
At the start: 2 copper layers, 39.6 x 29.5 mm, 17 parts, among them J1 Conn_01x03_Female, J2 Conn_01x02_Female, Q1 Q_NMOS_DGS, U1 NE555D

Commit message: Add files via upload
Parts:
- C1: value 10uF -> 100uF; footprint Capacitor_SMD:C_0805_2012Metric_Pad1.18x1.45mm_HandSolder -> Capacitor_Tantalum_SMD:CP_EIA-7343-31_Kemet-D_Pad2.25x2.55mm_HandSolder
- R3: value 0 -> 10k
- R4: value 5k -> 20k
- moved C1 2.54 mm to (147.2, 87.9)
Routing:
- net GND: track 19.0 -> 20.6 mm
- net Net-(R4-Pad2): track 16.5 -> 17.8 mm
